Commit message: feat(vslam): add small turtle urdf sensor prep

File: Robotics/VSLAM/trashbot_description/urdf/turtle_small.urdf.xacro (robot description, xacro)
@@ -1,45 +1,180 @@
 <?xml version="1.0"?>
 <robot xmlns:xacro="http://www.ros.org/wiki/xacro" name="turtle_small">
+  <xacro:property name="pi" value="3.141592653589793"/>
   <xacro:property name="mesh_file" value="package://trashbot_description/meshes/turtle_small_visual_mesh.stl"/>
-  <!-- Tunable sensor offsets (meters, radians) -->
-  <xacro:property name="camera_xyz" value="0 0 0"/>
-  <xacro:property name="camera_rpy" value="0 0 0"/>
-  <xacro:property name="imu_xyz" value="0 0 0"/>
-  <xacro:property name="imu_rpy" value="0 0 0"/>
-  <xacro:property name="gps_xyz" value="0 0 0"/>
-  <xacro:property name="gps_rpy" value="0 0 0"/>
-  <link name="base_link">
+  <!--
+    Small turtle tracked chassis first draft.
+    STL bounds check:
+      x = 0.1776 m
+      y = 0.1580 m
+      z = 0.0504 m
+    The exported mesh is centered in x/y and starts at z=0, so base_link is
+    placed at the chassis center height and the mesh/collision are shifted down
+    by half the chassis height.
+  -->
+  <xacro:property name="base_length" value="0.1776"/>
+  <xacro:property name="base_width" value="0.1580"/>
+  <xacro:property name="base_height" value="0.0504"/>
+  <xacro:property name="base_mass" value="6.0"/>
+  <xacro:property name="base_link_z" value="${base_height / 2.0}"/>
+  <!-- Collision stays simple even if the visual mesh includes tracks/sprockets. -->
+  <xacro:property name="collision_length" value="${base_length}"/>
+  <xacro:property name="collision_width" value="${base_width}"/>
+  <xacro:property name="collision_height" value="${base_height}"/>
+  <!-- Placeholder sensor offsets from base_link until the real mount is measured. -->
+  <xacro:property name="camera_x" value="0.060"/>
+  <xacro:property name="camera_y" value="0.0"/>
+  <xacro:property name="camera_z" value="0.040"/>
+  <xacro:property name="camera_roll" value="0.0"/>
+  <xacro:property name="camera_pitch" value="0.0"/>
+  <xacro:property name="camera_yaw" value="0.0"/>
+  <xacro:property name="imu_x" value="0.0"/>
+  <xacro:property name="imu_y" value="0.0"/>
+  <xacro:property name="imu_z" value="0.030"/>
+  <xacro:property name="imu_roll" value="0.0"/>
+  <xacro:property name="imu_pitch" value="0.0"/>
+  <xacro:property name="imu_yaw" value="0.0"/>
+  <xacro:property name="gps_x" value="-0.050"/>
+  <xacro:property name="gps_y" value="0.0"/>
+  <xacro:property name="gps_z" value="0.040"/>
+  <xacro:property name="gps_r" value="0.020"/>
+  <xacro:property name="gps_h" value="0.010"/>
+  <material name="chassis_gray">
+    <color rgba="0.55 0.55 0.58 1.0"/>
+  </material>
+  <material name="sensor_black">
+    <color rgba="0.02 0.02 0.02 1.0"/>
+  </material>
+  <material name="imu_green">
+    <color rgba="0.0 0.65 0.25 1.0"/>
+  </material>
+  <material name="gps_yellow">
+    <color rgba="0.95 0.75 0.1 1.0"/>
+  </material>
+  <xacro:macro name="box_inertial" params="mass x y z">
+    <inertial>
+      <mass value="${mass}"/>
+      <inertia
+        ixx="${mass * (y*y + z*z) / 12.0}"
+        ixy="0.0"
+        ixz="0.0"
+        iyy="${mass * (x*x + z*z) / 12.0}"
+        iyz="0.0"
+        izz="${mass * (x*x + y*y) / 12.0}"/>
+    </inertial>
+  </xacro:macro>
+  <xacro:macro name="cylinder_inertial" params="mass radius length">
+    <inertial>
+      <mass value="${mass}"/>
+      <inertia
+        ixx="${mass * (3.0 * radius * radius + length * length) / 12.0}"
+        ixy="0.0"
+        ixz="0.0"
+        iyy="${mass * radius * radius / 2.0}"
+        iyz="0.0"
+        izz="${mass * (3.0 * radius * radius + length * length) / 12.0}"/>
+    </inertial>
+  </xacro:macro>
+  <link name="base_footprint"/>
+  <link name="base_link"/>
+  <joint name="base_footprint_to_base_link" type="fixed">
+    <parent link="base_footprint"/>
+    <child link="base_link"/>
+    <origin xyz="0 0 ${base_link_z}" rpy="0 0 0"/>
+  </joint>
+  <link name="chassis_link">
     <visual>
+      <origin xyz="0 0 ${-base_height / 2.0}" rpy="0 0 0"/>
       <geometry>
         <mesh filename="${mesh_file}"/>
       </geometry>
+      <material name="chassis_gray"/>
+    </visual>
+    <collision>
+      <origin xyz="0 0 ${-collision_height / 2.0}" rpy="0 0 0"/>
+      <geometry>
+        <box size="${collision_length} ${collision_width} ${collision_height}"/>
+      </geometry>
+    </collision>
+    <xacro:box_inertial
+      mass="${base_mass}"
+      x="${collision_length}"
+      y="${collision_width}"
+      z="${collision_height}"/>
+  </link>
+  <joint name="base_to_chassis" type="fixed">
+    <parent link="base_link"/>
+    <child link="chassis_link"/>
+    <origin xyz="0 0 0" rpy="0 0 0"/>
+  </joint>
+  <link name="camera_link">
+    <visual>
+      <geometry>
+        <box size="0.09 0.025 0.025"/>
+      </geometry>
+      <material name="sensor_black"/>
     </visual>
     <collision>
       <geometry>
-        <box size="0.22 0.15 0.08"/>
+        <box size="0.09 0.025 0.025"/>
       </geometry>
     </collision>
-    <inertial>
-      <mass value="6.0"/>
-      <inertia ixx="0.06" ixy="0.0" ixz="0.0" iyy="0.06" iyz="0.0" izz="0.06"/>
-    </inertial>
+    <xacro:box_inertial mass="0.08" x="0.09" y="0.025" z="0.025"/>
   </link>
-  <link name="camera_link"/>
   <joint name="base_to_camera" type="fixed">
     <parent link="base_link"/>
     <child link="camera_link"/>
-    <origin xyz="${camera_xyz}" rpy="${camera_rpy}"/>
+    <origin xyz="${camera_x} ${camera_y} ${camera_z}" rpy="${camera_roll} ${camera_pitch} ${camera_yaw}"/>
   </joint>
-  <link name="imu_link"/>
+  <!-- D435i optical frame convention: z forward, x right, y down. -->
+  <link name="camera_color_optical_frame"/>
+  <joint name="camera_link_to_color_optical_frame" type="fixed">
+    <parent link="camera_link"/>
+    <child link="camera_color_optical_frame"/>
+    <origin xyz="0 0 0" rpy="${-pi / 2.0} 0 ${-pi / 2.0}"/>
+  </joint>
+  <link name="camera_depth_optical_frame"/>
+  <joint name="camera_link_to_depth_optical_frame" type="fixed">
+    <parent link="camera_link"/>
+    <child link="camera_depth_optical_frame"/>
+    <origin xyz="0 0 0" rpy="${-pi / 2.0} 0 ${-pi / 2.0}"/>
+  </joint>
+  <link name="imu_link">
+    <visual>
+      <geometry>
+        <box size="0.035 0.035 0.008"/>
+      </geometry>
+      <material name="imu_green"/>
+    </visual>
+    <collision>
+      <geometry>
+        <box size="0.035 0.035 0.008"/>
+      </geometry>
+    </collision>
+    <xacro:box_inertial mass="0.01" x="0.035" y="0.035" z="0.008"/>
+  </link>
   <joint name="base_to_imu" type="fixed">
     <parent link="base_link"/>
     <child link="imu_link"/>
-    <origin xyz="${imu_xyz}" rpy="${imu_rpy}"/>
+    <origin xyz="${imu_x} ${imu_y} ${imu_z}" rpy="${imu_roll} ${imu_pitch} ${imu_yaw}"/>
   </joint>
-  <link name="gps_link"/>
+  <link name="gps_link">
+    <visual>
+      <geometry>
+        <cylinder radius="${gps_r}" length="${gps_h}"/>
+      </geometry>
+      <material name="gps_yellow"/>
+    </visual>
+    <collision>
+      <geometry>
+        <cylinder radius="${gps_r}" length="${gps_h}"/>
+      </geometry>
+    </collision>
+    <xacro:cylinder_inertial mass="0.04" radius="${gps_r}" length="${gps_h}"/>
+  </link>
   <joint name="base_to_gps" type="fixed">
     <parent link="base_link"/>
     <child link="gps_link"/>
-    <origin xyz="${gps_xyz}" rpy="${gps_rpy}"/>
+    <origin xyz="${gps_x} ${gps_y} ${gps_z}" rpy="0 0 0"/>
   </joint>
 </robot>

Commit message: docs: record small turtle urdf planning

File: Robotics/VSLAM/trashbot_description/urdf/turtle_small.urdf.xacro (robot description, xacro)
@@ -22,20 +22,38 @@
   <xacro:property name="collision_width" value="${base_width}"/>
   <xacro:property name="collision_height" value="${base_height}"/>
-  <!-- Placeholder sensor offsets from base_link until the real mount is measured. -->
-  <xacro:property name="camera_x" value="0.060"/>
-  <xacro:property name="camera_y" value="0.0"/>
-  <xacro:property name="camera_z" value="0.040"/>
+  <!-- Tracked drive geometry first Onshape measurements. -->
+  <xacro:property name="track_width" value="0.137553"/>
+  <xacro:property name="half_track_width" value="${track_width / 2.0}"/>
+  <xacro:property name="effective_track_radius" value="0.021"/>
+  <!-- Actual asymmetric drive sprocket centers from base_link, kept as CAD reference. -->
+  <xacro:property name="left_drive_axis_x" value="-0.057871"/>
+  <xacro:property name="left_drive_axis_y" value="0.068776"/>
+  <xacro:property name="left_drive_axis_z" value="-0.000300"/>
+  <xacro:property name="right_drive_axis_x" value="0.058000"/>
+  <xacro:property name="right_drive_axis_y" value="-0.068777"/>
+  <xacro:property name="right_drive_axis_z" value="0.000000"/>
+  <!-- Initial diff-drive approximation uses aligned virtual wheels at x=0. -->
+  <xacro:property name="virtual_wheel_x" value="0.0"/>
+  <xacro:property name="left_virtual_wheel_y" value="${half_track_width}"/>
+  <xacro:property name="right_virtual_wheel_y" value="${-half_track_width}"/>
+  <xacro:property name="virtual_wheel_z" value="0.0"/>
+  <!-- D435i first Onshape measurement from base_link_mc to camera_link_mc. -->
+  <xacro:property name="camera_x" value="0.127688"/>
+  <xacro:property name="camera_y" value="-0.001695"/>
+  <xacro:property name="camera_z" value="0.107616"/>
   <xacro:property name="camera_roll" value="0.0"/>
   <xacro:property name="camera_pitch" value="0.0"/>
   <xacro:property name="camera_yaw" value="0.0"/>
-  <xacro:property name="imu_x" value="0.0"/>
-  <xacro:property name="imu_y" value="0.0"/>
-  <xacro:property name="imu_z" value="0.030"/>
+  <!-- BNO08x first Onshape measurement from base_link_mc to imu_link_mc. -->
+  <xacro:property name="imu_x" value="-0.010844"/>
+  <xacro:property name="imu_y" value="0.022228"/>
+  <xacro:property name="imu_z" value="0.018394"/>
   <xacro:property name="imu_roll" value="0.0"/>
   <xacro:property name="imu_pitch" value="0.0"/>
   <xacro:property name="imu_yaw" value="0.0"/>
-  <xacro:property name="gps_x" value="-0.050"/>
-  <xacro:property name="gps_y" value="0.0"/>
-  <xacro:property name="gps_z" value="0.040"/>
+  <!-- GPS first Onshape measurement from base_link_mc to gps_link_mc. -->
+  <xacro:property name="gps_x" value="-0.194160"/>
+  <xacro:property name="gps_y" value="-0.000001"/>
+  <xacro:property name="gps_z" value="0.037943"/>
   <xacro:property name="gps_r" value="0.020"/>
   <xacro:property name="gps_h" value="0.010"/>
