Commit message: feat: add Mari RViz TF checks and Jetson handoff

File: Robotics/VSLAM/trashbot_description/urdf/mari.urdf.xacro (robot description, xacro)
@@ -4,11 +4,11 @@
   <!--
     Mari tracked chassis first draft.
-    STL bounds check:
-      x = 0.1776 m
-      y = 0.1580 m
-      z = 0.0504 m
-    The exported mesh is centered in x/y and starts at z=0, so base_link is
-    placed at the chassis center height and the mesh/collision are shifted down
-    by half the chassis height.
+    Visual STL bounds check:
+      x = 0.5775 m
+      y = 0.5095 m
+      z = 0.1810 m
+      min_z = -0.021884 m
+    Keep base_footprint on the ground, base_link at the chassis center height,
+    and shift only the visual mesh so the lowest mesh vertex sits on z=0.
   -->
   <xacro:property name="base_length" value="0.1776"/>
@@ -17,4 +17,8 @@
   <xacro:property name="base_mass" value="6.0"/>
   <xacro:property name="base_link_z" value="${base_height / 2.0}"/>
+  <!-- Onshape STL export axis correction: keep ROS links fixed and rotate only the visual mesh. -->
+  <xacro:property name="chassis_mesh_yaw" value="${pi / 2.0}"/>
+  <xacro:property name="chassis_mesh_min_z" value="-0.021884"/>
+  <xacro:property name="chassis_mesh_z" value="${-base_link_z - chassis_mesh_min_z}"/>
   <!-- Collision stays simple even if the visual mesh includes tracks/sprockets. -->
   <xacro:property name="collision_length" value="${base_length}"/>
@@ -37,8 +41,9 @@
   <xacro:property name="right_virtual_wheel_y" value="${-half_track_width}"/>
   <xacro:property name="virtual_wheel_z" value="0.0"/>
-  <!-- D435i first Onshape measurement from base_link_mc to camera_link_mc. -->
+  <!-- D435i mount measurement from base_link_mc to camera_link_mc.
+       2026-04-27: camera height raised by (80 - 65.44216) mm = 0.01455784 m. -->
   <xacro:property name="camera_x" value="0.127688"/>
   <xacro:property name="camera_y" value="-0.001695"/>
-  <xacro:property name="camera_z" value="0.107616"/>
+  <xacro:property name="camera_z" value="0.122174"/>
   <xacro:property name="camera_roll" value="0.0"/>
   <xacro:property name="camera_pitch" value="0.0"/>
@@ -102,5 +107,5 @@
   <link name="chassis_link">
     <visual>
-      <origin xyz="0 0 ${-base_height / 2.0}" rpy="0 0 0"/>
+      <origin xyz="0 0 ${chassis_mesh_z}" rpy="0 0 ${chassis_mesh_yaw}"/>
       <geometry>
         <mesh filename="${mesh_file}"/>
@@ -109,5 +114,5 @@
     </visual>
     <collision>
-      <origin xyz="0 0 ${-collision_height / 2.0}" rpy="0 0 0"/>
+      <origin xyz="0 0 0" rpy="0 0 0"/>
       <geometry>
         <box size="${collision_length} ${collision_width} ${collision_height}"/>
@@ -128,5 +133,5 @@
     <visual>
       <geometry>
-        <box size="0.09 0.025 0.025"/>
+        <box size="0.025 0.09 0.025"/>
       </geometry>
       <material name="sensor_black"/>
@@ -134,8 +139,8 @@
     <collision>
       <geometry>
-        <box size="0.09 0.025 0.025"/>
-      </geometry>
-    </collision>
-    <xacro:box_inertial mass="0.08" x="0.09" y="0.025" z="0.025"/>
+        <box size="0.025 0.09 0.025"/>
+      </geometry>
+    </collision>
+    <xacro:box_inertial mass="0.08" x="0.025" y="0.09" z="0.025"/>
   </link>
   <joint name="base_to_camera" type="fixed">

Commit message: feat(vslam): add Mari Gazebo RTAB-Map baseline

File: Robotics/VSLAM/trashbot_description/urdf/mari.urdf.xacro (robot description, xacro)
@@ -1,4 +1,5 @@
 <?xml version="1.0"?>
 <robot xmlns:xacro="http://www.ros.org/wiki/xacro" name="mari">
+  <xacro:arg name="use_mesh_visual" default="true"/>
   <xacro:property name="mesh_file" value="package://trashbot_description/meshes/mari_visual_mesh.stl"/>
   <!--
@@ -9,6 +10,6 @@
       z = 0.1810 m
       min_z = -0.021884 m
-    Keep base_footprint on the ground, base_link at the chassis center height,
-    and shift only the visual mesh so the lowest mesh vertex sits on z=0.
+    Keep base_footprint on the ground, base_link at the STL chassis center
+    height, and shift only the visual mesh so the lowest mesh vertex sits on z=0.
   -->
   <xacro:property name="base_length" value="0.1776"/>
@@ -25,4 +26,5 @@
   <xacro:property name="collision_width" value="${base_width}"/>
   <xacro:property name="collision_height" value="${base_height}"/>
+  <xacro:property name="collision_z" value="0.012"/>
   <!-- Tracked drive geometry first Onshape measurements. -->
   <xacro:property name="track_width" value="0.137553"/>
@@ -36,17 +38,33 @@
   <xacro:property name="right_drive_axis_y" value="-0.068777"/>
   <xacro:property name="right_drive_axis_z" value="0.000000"/>
-  <!-- Initial diff-drive approximation uses aligned virtual wheels at x=0. -->
-  <xacro:property name="virtual_wheel_x" value="0.0"/>
-  <xacro:property name="left_virtual_wheel_y" value="${half_track_width}"/>
-  <xacro:property name="right_virtual_wheel_y" value="${-half_track_width}"/>
-  <xacro:property name="virtual_wheel_z" value="0.0"/>
+  <!--
+    Gazebo tracked-contact approximation.
+    The STL already shows the tracks; these four collision-only wheels provide
+    front/rear support. The /cmd_vel controller below uses planar movement so
+    simulation control remains stable while real encoder validation stays
+    hardware-topic based.
+  -->
+  <xacro:property name="track_contact_x_offset" value="0.058"/>
+  <xacro:property name="front_track_wheel_x" value="${track_contact_x_offset}"/>
+  <xacro:property name="rear_track_wheel_x" value="${-track_contact_x_offset}"/>
+  <xacro:property name="left_track_wheel_y" value="${half_track_width}"/>
+  <xacro:property name="right_track_wheel_y" value="${-half_track_width}"/>
+  <xacro:property name="virtual_wheel_z" value="${effective_track_radius - base_link_z}"/>
+  <xacro:property name="virtual_wheel_width" value="0.014"/>
+  <xacro:property name="virtual_wheel_mass" value="0.08"/>
   <!-- D435i mount measurement from base_link_mc to camera_link_mc.
-       2026-04-27: camera height raised by (80 - 65.44216) mm = 0.01455784 m. -->
+       2026-04-28: lowered 10 mm from the 2026-04-27 0.122174 m reference. -->
   <xacro:property name="camera_x" value="0.127688"/>
   <xacro:property name="camera_y" value="-0.001695"/>
-  <xacro:property name="camera_z" value="0.122174"/>
+  <xacro:property name="camera_z" value="0.112174"/>
   <xacro:property name="camera_roll" value="0.0"/>
   <xacro:property name="camera_pitch" value="0.0"/>
   <xacro:property name="camera_yaw" value="0.0"/>
+  <xacro:property name="sim_camera_update_rate" value="15.0"/>
+  <xacro:property name="sim_camera_width" value="640"/>
+  <xacro:property name="sim_camera_height" value="480"/>
+  <xacro:property name="sim_camera_horizontal_fov" value="1.3962634"/>
+  <xacro:property name="sim_camera_near_clip" value="0.10"/>
+  <xacro:property name="sim_camera_far_clip" value="6.00"/>
   <!-- BNO08x first Onshape measurement from base_link_mc to imu_link_mc. -->
   <xacro:property name="imu_x" value="-0.010844"/>
@@ -56,4 +74,5 @@
   <xacro:property name="imu_pitch" value="0.0"/>
   <xacro:property name="imu_yaw" value="0.0"/>
+  <xacro:property name="sim_imu_update_rate" value="100.0"/>
   <!-- GPS first Onshape measurement from base_link_mc to gps_link_mc. -->
   <xacro:property name="gps_x" value="-0.194160"/>
@@ -73,4 +92,7 @@
   <material name="gps_yellow">
     <color rgba="0.95 0.75 0.1 1.0"/>
+  </material>
+  <material name="virtual_wheel_dark">
+    <color rgba="0.03 0.03 0.03 1.0"/>
   </material>
   <xacro:macro name="box_inertial" params="mass x y z">
@@ -98,4 +120,24 @@
     </inertial>
   </xacro:macro>
+  <xacro:macro name="virtual_track_wheel" params="prefix x y">
+    <link name="${prefix}_virtual_track_wheel_link">
+      <collision>
+        <origin xyz="0 0 0" rpy="${pi / 2.0} 0 0"/>
+        <geometry>
+          <cylinder radius="${effective_track_radius}" length="${virtual_wheel_width}"/>
+        </geometry>
+      </collision>
+      <xacro:cylinder_inertial
+        mass="${virtual_wheel_mass}"
+        radius="${effective_track_radius}"
+        length="${virtual_wheel_width}"/>
+    </link>
+    <joint name="${prefix}_virtual_track_wheel_joint" type="continuous">
+      <parent link="base_link"/>
+      <child link="${prefix}_virtual_track_wheel_link"/>
+      <origin xyz="${x} ${y} ${virtual_wheel_z}" rpy="0 0 0"/>
+      <axis xyz="0 1 0"/>
+    </joint>
+  </xacro:macro>
   <link name="base_footprint"/>
   <link name="base_link"/>
@@ -106,5 +148,6 @@
   </joint>
   <link name="chassis_link">
-    <visual>
+    <visual name="mesh_visual">
+      <xacro:if value="$(arg use_mesh_visual)">
       <origin xyz="0 0 ${chassis_mesh_z}" rpy="0 0 ${chassis_mesh_yaw}"/>
       <geometry>
@@ -112,7 +155,15 @@
       </geometry>
       <material name="chassis_gray"/>
+      </xacro:if>
+      <xacro:unless value="$(arg use_mesh_visual)">
+      <origin xyz="0 0 0" rpy="0 0 0"/>
+      <geometry>
+        <box size="${base_length} ${base_width} ${base_height}"/>
+      </geometry>
+      <material name="chassis_gray"/>
+      </xacro:unless>
     </visual>
     <collision>
-      <origin xyz="0 0 0" rpy="0 0 0"/>
+      <origin xyz="0 0 ${collision_z}" rpy="0 0 0"/>
       <geometry>
         <box size="${collision_length} ${collision_width} ${collision_height}"/>
@@ -130,4 +181,8 @@
     <origin xyz="0 0 0" rpy="0 0 0"/>
   </joint>
+  <xacro:virtual_track_wheel prefix="left_front" x="${front_track_wheel_x}" y="${left_track_wheel_y}"/>
+  <xacro:virtual_track_wheel prefix="right_front" x="${front_track_wheel_x}" y="${right_track_wheel_y}"/>
+  <xacro:virtual_track_wheel prefix="left_rear" x="${rear_track_wheel_x}" y="${left_track_wheel_y}"/>
+  <xacro:virtual_track_wheel prefix="right_rear" x="${rear_track_wheel_x}" y="${right_track_wheel_y}"/>
   <link name="camera_link">
     <visual>
@@ -200,3 +255,137 @@
     <origin xyz="${gps_x} ${gps_y} ${gps_z}" rpy="0 0 0"/>
   </joint>
+  <gazebo reference="left_front_virtual_track_wheel_link">
+    <material>Gazebo/DarkGrey</material>
+    <mu1>0.2</mu1>
+    <mu2>0.2</mu2>
+  </gazebo>
+  <gazebo reference="right_front_virtual_track_wheel_link">
+    <material>Gazebo/DarkGrey</material>
+    <mu1>0.2</mu1>
+    <mu2>0.2</mu2>
+  </gazebo>
+  <gazebo reference="left_rear_virtual_track_wheel_link">
+    <material>Gazebo/DarkGrey</material>
+    <mu1>0.2</mu1>
+    <mu2>0.2</mu2>
+  </gazebo>
+  <gazebo reference="right_rear_virtual_track_wheel_link">
+    <material>Gazebo/DarkGrey</material>
+    <mu1>0.2</mu1>
+    <mu2>0.2</mu2>
+  </gazebo>
+  <gazebo reference="imu_link">
+    <sensor name="mari_imu" type="imu">
+      <always_on>true</always_on>
+      <update_rate>${sim_imu_update_rate}</update_rate>
+      <visualize>false</visualize>
+      <imu>
+        <angular_velocity>
+          <x>
+            <noise type="gaussian">
+              <mean>0.0</mean>
+              <stddev>0.0002</stddev>
+            </noise>
+          </x>
+          <y>
+            <noise type="gaussian">
+              <mean>0.0</mean>
+              <stddev>0.0002</stddev>
+            </noise>
+          </y>
+          <z>
+            <noise type="gaussian">
+              <mean>0.0</mean>
+              <stddev>0.0002</stddev>
+            </noise>
+          </z>
+        </angular_velocity>
+        <linear_acceleration>
+          <x>
+            <noise type="gaussian">
+              <mean>0.0</mean>
+              <stddev>0.01</stddev>
+            </noise>
+          </x>
+          <y>
+            <noise type="gaussian">
+              <mean>0.0</mean>
+              <stddev>0.01</stddev>
+            </noise>
+          </y>
+          <z>
+            <noise type="gaussian">
+              <mean>0.0</mean>
+              <stddev>0.01</stddev>
+            </noise>
+          </z>
+        </linear_acceleration>
+      </imu>
+      <plugin name="mari_imu_sensor" filename="libgazebo_ros_imu_sensor.so">
+        <initial_orientation_as_reference>false</initial_orientation_as_reference>
+        <frame_name>imu_link</frame_name>
+        <ros>
+          <remapping>~/out:=/imu/data</remapping>
+        </ros>
+      </plugin>
+    </sensor>
+  </gazebo>
+  <gazebo reference="camera_link">
+    <sensor name="mari_rgbd_camera" type="depth">
+      <always_on>true</always_on>
+      <update_rate>${sim_camera_update_rate}</update_rate>
+      <visualize>true</visualize>
+      <camera name="mari_rgbd_camera_optics">
+        <horizontal_fov>${sim_camera_horizontal_fov}</horizontal_fov>
+        <image>
+          <width>${sim_camera_width}</width>
+          <height>${sim_camera_height}</height>
+          <format>R8G8B8</format>
+        </image>
+        <depth_camera>
+        </depth_camera>
+        <clip>
+          <near>${sim_camera_near_clip}</near>
+          <far>${sim_camera_far_clip}</far>
+        </clip>
+        <noise>
+          <type>gaussian</type>
+          <mean>0.0</mean>
+          <stddev>0.005</stddev>
+        </noise>
+      </camera>
+      <plugin name="mari_rgbd_camera_controller" filename="libgazebo_ros_camera.so">
+        <ros>
+          <remapping>camera/image_raw:=/camera/camera/color/image_raw</remapping>
+          <remapping>camera/camera_info:=/camera/camera/color/camera_info</remapping>
+          <remapping>camera/depth/image_raw:=/camera/camera/aligned_depth_to_color/image_raw</remapping>
+          <remapping>camera/depth/camera_info:=/camera/camera/aligned_depth_to_color/camera_info</remapping>
+          <remapping>camera/points:=/camera/camera/depth/color/points</remapping>
+        </ros>
+        <camera_name>camera</camera_name>
+        <frame_name>camera_color_optical_frame</frame_name>
+        <hack_baseline>0.0</hack_baseline>
+        <min_depth>${sim_camera_near_clip}</min_depth>
+        <max_depth>${sim_camera_far_clip}</max_depth>
+      </plugin>
+    </sensor>
+  </gazebo>
+  <gazebo>
+    <plugin name="mari_planar_move" filename="libgazebo_ros_planar_move.so">
+      <ros>
+        <remapping>/tf:=tf</remapping>
+      </ros>
+      <update_rate>100</update_rate>
+      <publish_rate>50</publish_rate>
+      <command_topic>cmd_vel</command_topic>
+      <odometry_topic>odom</odometry_topic>
+      <odometry_frame>odom</odometry_frame>
+      <robot_base_frame>base_footprint</robot_base_frame>
+      <publish_odom>true</publish_odom>
+      <publish_odom_tf>true</publish_odom_tf>
+      <covariance_x>0.0001</covariance_x>
+      <covariance_y>0.0001</covariance_y>
+      <covariance_yaw>0.01</covariance_yaw>
+    </plugin>
+  </gazebo>
 </robot>

Commit message: feat: add Mari Gazebo localization validation
Add Mari Gazebo sensor, encoder, EKF, RTAB-Map, park-world validation assets and documentation.

File: Robotics/VSLAM/trashbot_description/urdf/mari.urdf.xacro (robot description, xacro)
@@ -2,4 +2,8 @@
 <robot xmlns:xacro="http://www.ros.org/wiki/xacro" name="mari">
   <xacro:arg name="use_mesh_visual" default="true"/>
+  <xacro:arg name="sim_camera_update_rate" default="15.0"/>
+  <xacro:arg name="sim_camera_width" default="640"/>
+  <xacro:arg name="sim_camera_height" default="480"/>
+  <xacro:arg name="sim_camera_visualize" default="true"/>
   <xacro:property name="mesh_file" value="package://trashbot_description/meshes/mari_visual_mesh.stl"/>
   <!--
@@ -61,7 +65,4 @@
   <xacro:property name="camera_pitch" value="0.0"/>
   <xacro:property name="camera_yaw" value="0.0"/>
-  <xacro:property name="sim_camera_update_rate" value="15.0"/>
-  <xacro:property name="sim_camera_width" value="640"/>
-  <xacro:property name="sim_camera_height" value="480"/>
   <xacro:property name="sim_camera_horizontal_fov" value="1.3962634"/>
   <xacro:property name="sim_camera_near_clip" value="0.10"/>
@@ -81,4 +82,5 @@
   <xacro:property name="gps_r" value="0.020"/>
   <xacro:property name="gps_h" value="0.010"/>
+  <xacro:property name="sim_gps_update_rate" value="5.0"/>
   <material name="chassis_gray">
     <color rgba="0.55 0.55 0.58 1.0"/>
@@ -334,11 +336,11 @@
     <sensor name="mari_rgbd_camera" type="depth">
       <always_on>true</always_on>
-      <update_rate>${sim_camera_update_rate}</update_rate>
-      <visualize>true</visualize>
+      <update_rate>$(arg sim_camera_update_rate)</update_rate>
+      <visualize>$(arg sim_camera_visualize)</visualize>
       <camera name="mari_rgbd_camera_optics">
         <horizontal_fov>${sim_camera_horizontal_fov}</horizontal_fov>
         <image>
-          <width>${sim_camera_width}</width>
-          <height>${sim_camera_height}</height>
+          <width>$(arg sim_camera_width)</width>
+          <height>$(arg sim_camera_height)</height>
           <format>R8G8B8</format>
         </image>
@@ -371,4 +373,34 @@
     </sensor>
   </gazebo>
+  <gazebo reference="gps_link">
+    <sensor name="mari_gps" type="gps">
+      <always_on>true</always_on>
+      <update_rate>${sim_gps_update_rate}</update_rate>
+      <visualize>false</visualize>
+      <gps>
+        <position_sensing>
+          <horizontal>
+            <noise type="gaussian">
+              <mean>0.0</mean>
+              <stddev>0.0002</stddev>
+            </noise>
+          </horizontal>
+          <vertical>
+            <noise type="gaussian">
+              <mean>0.0</mean>
+              <stddev>0.0002</stddev>
+            </noise>
+          </vertical>
+        </position_sensing>
+      </gps>
+      <plugin name="mari_gps_sensor" filename="libgazebo_ros_gps_sensor.so">
+        <ros>
+          <namespace>/gps</namespace>
+          <remapping>~/out:=fix</remapping>
+          <remapping>~/vel:=velocity</remapping>
+        </ros>
+      </plugin>
+    </sensor>
+  </gazebo>
   <gazebo>
     <plugin name="mari_planar_move" filename="libgazebo_ros_planar_move.so">
