Commit message: docs(vslam): record S14P31C205-735 Duri validation

File: Robotics/VSLAM/trashbot_description/urdf/duri.urdf.xacro (robot description, xacro)
@@ -1,45 +1,327 @@
 <?xml version="1.0"?>
 <robot xmlns:xacro="http://www.ros.org/wiki/xacro" name="duri">
-  <xacro:property name="mesh_file" value="package://trashbot_description/meshes/duri_visual_mesh.stl"/>
-  <!-- Tunable sensor offsets (meters, radians) -->
-  <xacro:property name="camera_xyz" value="0 0 0"/>
-  <xacro:property name="camera_rpy" value="0 0 0"/>
-  <xacro:property name="imu_xyz" value="0 0 0"/>
-  <xacro:property name="imu_rpy" value="0 0 0"/>
-  <xacro:property name="gps_xyz" value="0 0 0"/>
-  <xacro:property name="gps_rpy" value="0 0 0"/>
-  <link name="base_link">
-    <visual>
-      <geometry>
-        <mesh filename="${mesh_file}"/>
-      </geometry>
+  <xacro:arg name="use_mesh_visual" default="true"/>
+  <xacro:arg name="sim_camera_update_rate" default="15.0"/>
+  <xacro:arg name="sim_camera_width" default="424"/>
+  <xacro:arg name="sim_camera_height" default="240"/>
+  <xacro:arg name="sim_camera_visualize" default="false"/>
+  <xacro:arg name="mesh_file" default="package://trashbot_description/meshes/duri_visual_mesh.stl"/>
+  <xacro:property name="visual_mesh_file" value="$(arg mesh_file)"/>
+  <!--
+    Duri tracked chassis first draft.
+    Onshape mate connector measurements were recorded in millimeters on 2026-05-08
+    and converted to meters here.
+  -->
+  <xacro:property name="base_length" value="0.62"/>
+  <xacro:property name="base_width" value="0.32"/>
+  <xacro:property name="base_height" value="0.18"/>
+  <xacro:property name="base_mass" value="12.0"/>
+  <xacro:property name="base_link_z" value="0.038536"/>
+  <xacro:property name="chassis_mesh_z" value="0.0"/>
+  <xacro:property name="chassis_mesh_yaw" value="${pi / 2.0}"/>
+  <!-- Keep collision simple; detailed turtle shell and track meshes are visual only. -->
+  <xacro:property name="collision_length" value="${base_length}"/>
+  <xacro:property name="collision_width" value="${base_width}"/>
+  <xacro:property name="collision_height" value="${2.0 * base_link_z}"/>
+  <xacro:property name="collision_z" value="0.0"/>
+  <!-- Duri-specific sensor mount measurements from base_link_mc. -->
+  <xacro:property name="camera_x" value="0.245385"/>
+  <xacro:property name="camera_y" value="0.0"/>
+  <xacro:property name="camera_z" value="0.120895"/>
+  <xacro:property name="camera_roll" value="0.0"/>
+  <xacro:property name="camera_pitch" value="0.0"/>
+  <xacro:property name="camera_yaw" value="0.0"/>
+  <xacro:property name="sim_camera_horizontal_fov" value="1.3962634"/>
+  <xacro:property name="sim_camera_near_clip" value="0.10"/>
+  <xacro:property name="sim_camera_far_clip" value="6.00"/>
+  <xacro:property name="imu_x" value="0.010724"/>
+  <xacro:property name="imu_y" value="-0.001608"/>
+  <xacro:property name="imu_z" value="0.089039"/>
+  <xacro:property name="imu_roll" value="0.0"/>
+  <xacro:property name="imu_pitch" value="0.0"/>
+  <xacro:property name="imu_yaw" value="0.0"/>
+  <xacro:property name="sim_imu_update_rate" value="100.0"/>
+  <xacro:property name="gps_x" value="-0.276881"/>
+  <xacro:property name="gps_y" value="0.0"/>
+  <xacro:property name="gps_z" value="0.005984"/>
+  <xacro:property name="gps_r" value="0.020"/>
+  <xacro:property name="gps_h" value="0.010"/>
+  <!-- Track ground-contact reference points from base_link_mc. -->
+  <xacro:property name="track_contact_z" value="-0.038536"/>
+  <xacro:property name="track_center_y" value="0.109858"/>
+  <xacro:property name="track_separation" value="${2.0 * track_center_y}"/>
+  <material name="chassis_gray">
+    <color rgba="0.55 0.55 0.58 1.0"/>
+  </material>
+  <material name="sensor_black">
+    <color rgba="0.02 0.02 0.02 1.0"/>
+  </material>
+  <material name="imu_green">
+    <color rgba="0.0 0.65 0.25 1.0"/>
+  </material>
+  <material name="gps_yellow">
+    <color rgba="0.95 0.75 0.1 1.0"/>
+  </material>
+  <xacro:macro name="box_inertial" params="mass x y z">
+    <inertial>
+      <mass value="${mass}"/>
+      <inertia
+        ixx="${mass * (y*y + z*z) / 12.0}"
+        ixy="0.0"
+        ixz="0.0"
+        iyy="${mass * (x*x + z*z) / 12.0}"
+        iyz="0.0"
+        izz="${mass * (x*x + y*y) / 12.0}"/>
+    </inertial>
+  </xacro:macro>
+  <xacro:macro name="cylinder_inertial" params="mass radius length">
+    <inertial>
+      <mass value="${mass}"/>
+      <inertia
+        ixx="${mass * (3.0 * radius * radius + length * length) / 12.0}"
+        ixy="0.0"
+        ixz="0.0"
+        iyy="${mass * radius * radius / 2.0}"
+        iyz="0.0"
+        izz="${mass * (3.0 * radius * radius + length * length) / 12.0}"/>
+    </inertial>
+  </xacro:macro>
+  <link name="base_footprint"/>
+  <link name="base_link"/>
+  <joint name="base_footprint_to_base_link" type="fixed">
+    <parent link="base_footprint"/>
+    <child link="base_link"/>
+    <origin xyz="0 0 ${base_link_z}" rpy="0 0 0"/>
+  </joint>
+  <link name="chassis_link">
+    <visual name="mesh_visual">
+      <xacro:if value="$(arg use_mesh_visual)">
+      <origin xyz="0 0 ${chassis_mesh_z}" rpy="0 0 ${chassis_mesh_yaw}"/>
+      <geometry>
+        <mesh filename="${visual_mesh_file}"/>
+      </geometry>
+      <material name="chassis_gray"/>
+      </xacro:if>
+      <xacro:unless value="$(arg use_mesh_visual)">
+      <origin xyz="0 0 ${collision_z}" rpy="0 0 0"/>
+      <geometry>
+        <box size="${collision_length} ${collision_width} ${collision_height}"/>
+      </geometry>
+      <material name="chassis_gray"/>
+      </xacro:unless>
     </visual>
     <collision>
-      <geometry>
-        <box size="0.30 0.20 0.10"/>
+      <origin xyz="0 0 ${collision_z}" rpy="0 0 0"/>
+      <geometry>
+        <box size="${collision_length} ${collision_width} ${collision_height}"/>
       </geometry>
     </collision>
-    <inertial>
-      <mass value="10.0"/>
-      <inertia ixx="0.1" ixy="0.0" ixz="0.0" iyy="0.1" iyz="0.0" izz="0.1"/>
-    </inertial>
+    <xacro:box_inertial
+      mass="${base_mass}"
+      x="${collision_length}"
+      y="${collision_width}"
+      z="${collision_height}"/>
   </link>
-  <link name="camera_link"/>
+  <joint name="base_to_chassis" type="fixed">
+    <parent link="base_link"/>
+    <child link="chassis_link"/>
+    <origin xyz="0 0 0" rpy="0 0 0"/>
+  </joint>
+  <link name="camera_link">
+    <visual>
+      <geometry>
+        <box size="0.025 0.09 0.025"/>
+      </geometry>
+      <material name="sensor_black"/>
+    </visual>
+    <collision>
+      <geometry>
+        <box size="0.025 0.09 0.025"/>
+      </geometry>
+    </collision>
+    <xacro:box_inertial mass="0.08" x="0.025" y="0.09" z="0.025"/>
+  </link>
   <joint name="base_to_camera" type="fixed">
     <parent link="base_link"/>
     <child link="camera_link"/>
-    <origin xyz="${camera_xyz}" rpy="${camera_rpy}"/>
-  </joint>
-  <link name="imu_link"/>
+    <origin xyz="${camera_x} ${camera_y} ${camera_z}" rpy="${camera_roll} ${camera_pitch} ${camera_yaw}"/>
+  </joint>
+  <!-- D435i optical frame convention: z forward, x right, y down. -->
+  <link name="camera_color_optical_frame"/>
+  <joint name="camera_link_to_color_optical_frame" type="fixed">
+    <parent link="camera_link"/>
+    <child link="camera_color_optical_frame"/>
+    <origin xyz="0 0 0" rpy="${-pi / 2.0} 0 ${-pi / 2.0}"/>
+  </joint>
+  <link name="camera_depth_optical_frame"/>
+  <joint name="camera_link_to_depth_optical_frame" type="fixed">
+    <parent link="camera_link"/>
+    <child link="camera_depth_optical_frame"/>
+    <origin xyz="0 0 0" rpy="${-pi / 2.0} 0 ${-pi / 2.0}"/>
+  </joint>
+  <link name="imu_link">
+    <visual>
+      <geometry>
+        <box size="0.035 0.035 0.008"/>
+      </geometry>
+      <material name="imu_green"/>
+    </visual>
+    <collision>
+      <geometry>
+        <box size="0.035 0.035 0.008"/>
+      </geometry>
+    </collision>
+    <xacro:box_inertial mass="0.01" x="0.035" y="0.035" z="0.008"/>
+  </link>
   <joint name="base_to_imu" type="fixed">
     <parent link="base_link"/>
     <child link="imu_link"/>
-    <origin xyz="${imu_xyz}" rpy="${imu_rpy}"/>
-  </joint>
-  <link name="gps_link"/>
+    <origin xyz="${imu_x} ${imu_y} ${imu_z}" rpy="${imu_roll} ${imu_pitch} ${imu_yaw}"/>
+  </joint>
+  <link name="gps_link">
+    <visual>
+      <geometry>
+        <cylinder radius="${gps_r}" length="${gps_h}"/>
+      </geometry>
+      <material name="gps_yellow"/>
+    </visual>
+    <collision>
+      <geometry>
+        <cylinder radius="${gps_r}" length="${gps_h}"/>
+      </geometry>
+    </collision>
+    <xacro:cylinder_inertial mass="0.04" radius="${gps_r}" length="${gps_h}"/>
+  </link>
   <joint name="base_to_gps" type="fixed">
     <parent link="base_link"/>
     <child link="gps_link"/>
-    <origin xyz="${gps_xyz}" rpy="${gps_rpy}"/>
-  </joint>
+    <origin xyz="${gps_x} ${gps_y} ${gps_z}" rpy="0 0 0"/>
+  </joint>
+  <!-- Empty reference links for future Gazebo/odometry track geometry checks. -->
+  <link name="track_left_contact_link"/>
+  <joint name="base_to_track_left_contact" type="fixed">
+    <parent link="base_link"/>
+    <child link="track_left_contact_link"/>
+    <origin xyz="0 ${track_center_y} ${track_contact_z}" rpy="0 0 0"/>
+  </joint>
+  <link name="track_right_contact_link"/>
+  <joint name="base_to_track_right_contact" type="fixed">
+    <parent link="base_link"/>
+    <child link="track_right_contact_link"/>
+    <origin xyz="0 ${-track_center_y} ${track_contact_z}" rpy="0 0 0"/>
+  </joint>
+  <gazebo reference="imu_link">
+    <sensor name="duri_imu" type="imu">
+      <always_on>true</always_on>
+      <update_rate>${sim_imu_update_rate}</update_rate>
+      <visualize>false</visualize>
+      <imu>
+        <angular_velocity>
+          <x>
+            <noise type="gaussian">
+              <mean>0.0</mean>
+              <stddev>0.0002</stddev>
+            </noise>
+          </x>
+          <y>
+            <noise type="gaussian">
+              <mean>0.0</mean>
+              <stddev>0.0002</stddev>
+            </noise>
+          </y>
+          <z>
+            <noise type="gaussian">
+              <mean>0.0</mean>
+              <stddev>0.0002</stddev>
+            </noise>
+          </z>
+        </angular_velocity>
+        <linear_acceleration>
+          <x>
+            <noise type="gaussian">
+              <mean>0.0</mean>
+              <stddev>0.01</stddev>
+            </noise>
+          </x>
+          <y>
+            <noise type="gaussian">
+              <mean>0.0</mean>
+              <stddev>0.01</stddev>
+            </noise>
+          </y>
+          <z>
+            <noise type="gaussian">
+              <mean>0.0</mean>
+              <stddev>0.01</stddev>
+            </noise>
+          </z>
+        </linear_acceleration>
+      </imu>
+      <plugin name="duri_imu_sensor" filename="libgazebo_ros_imu_sensor.so">
+        <initial_orientation_as_reference>false</initial_orientation_as_reference>
+        <frame_name>imu_link</frame_name>
+        <ros>
+          <remapping>~/out:=/imu/data</remapping>
+        </ros>
+      </plugin>
+    </sensor>
+  </gazebo>
+  <gazebo reference="camera_link">
+    <sensor name="duri_rgbd_camera" type="depth">
+      <always_on>true</always_on>
+      <update_rate>$(arg sim_camera_update_rate)</update_rate>
+      <visualize>$(arg sim_camera_visualize)</visualize>
+      <camera name="duri_rgbd_camera_optics">
+        <horizontal_fov>${sim_camera_horizontal_fov}</horizontal_fov>
+        <image>
+          <width>$(arg sim_camera_width)</width>
+          <height>$(arg sim_camera_height)</height>
+          <format>R8G8B8</format>
+        </image>
+        <depth_camera>
+        </depth_camera>
+        <clip>
+          <near>${sim_camera_near_clip}</near>
+          <far>${sim_camera_far_clip}</far>
+        </clip>
+        <noise>
+          <type>gaussian</type>
+          <mean>0.0</mean>
+          <stddev>0.005</stddev>
+        </noise>
+      </camera>
+      <plugin name="duri_rgbd_camera_controller" filename="libgazebo_ros_camera.so">
+        <ros>
+          <remapping>camera/image_raw:=/camera/camera/color/image_raw</remapping>
+          <remapping>camera/camera_info:=/camera/camera/color/camera_info</remapping>
+          <remapping>camera/depth/image_raw:=/camera/camera/aligned_depth_to_color/image_raw</remapping>
+          <remapping>camera/depth/camera_info:=/camera/camera/aligned_depth_to_color/camera_info</remapping>
+          <remapping>camera/points:=/camera/camera/depth/color/points</remapping>
+        </ros>
+        <camera_name>camera</camera_name>
+        <frame_name>camera_color_optical_frame</frame_name>
+        <hack_baseline>0.0</hack_baseline>
+        <min_depth>${sim_camera_near_clip}</min_depth>
+        <max_depth>${sim_camera_far_clip}</max_depth>
+      </plugin>
+    </sensor>
+  </gazebo>
+  <gazebo>
+    <plugin name="duri_planar_move" filename="libgazebo_ros_planar_move.so">
+      <ros>
+        <remapping>/tf:=tf</remapping>
+      </ros>
+      <update_rate>100</update_rate>
+      <publish_rate>50</publish_rate>
+      <command_topic>cmd_vel</command_topic>
+      <odometry_topic>odom</odometry_topic>
+      <odometry_frame>odom</odometry_frame>
+      <robot_base_frame>base_footprint</robot_base_frame>
+      <publish_odom>true</publish_odom>
+      <publish_odom_tf>true</publish_odom_tf>
+      <covariance_x>0.0001</covariance_x>
+      <covariance_y>0.0001</covariance_y>
+      <covariance_yaw>0.01</covariance_yaw>
+    </plugin>
+  </gazebo>
 </robot>
